File: RTL8019.sch (KiCad schematic (older format))
At the start: 54 parts, among them J1 ROM_0, J10 IRQ_2, J11 IO_0, J12 IO_1, J13 IO_2, J14 IO_3, J2 ROM_1, J3 ROM_2, J4 ROM_3, J5 ROM_4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

Commit message: Add files via upload
Fixed - incorrect rtl8019as footprint
Parts:
- R2, R3: value 220 -> 510
- U1: footprint Package_QFP:PQFP-100_14x20mm_P0.65mm -> 20f001ng:8019as
- X0: symbol Connector:Bus_ISA_8bit -> RTL8019-rescue:Bus_ISA_8bit-Connector
Changed lines of the file:
@@
 EESchema Schematic File Version 4
-LIBS:RTL8019-cache
 EELAYER 30 0
 EELAYER END
@@
 F 0 "U1" H 8944 3546 50  0000 L CNN
 F 1 "RTL8019AS" H 8944 3455 50  0000 L CNN
-F 2 "Package_QFP:PQFP-100_14x20mm_P0.65mm" H 6800 3450 50  0001 C CNN
+F 2 "20f001ng:8019as" H 6800 3450 50  0001 C CNN
 F 3 "" H 6800 3450 50  0001 C CNN
 	1    6800 3450
@@
 NoConn ~ 7100 1850
 $Comp
-L Device:R R2
-U 1 1 5E84BDBA
-P 10550 7500
-F 0 "R2" H 10620 7546 50  0000 L CNN
-F 1 "220" H 10620 7455 50  0000 L CNN
-F 2 "Resistor_SMD:R_0805_2012Metric" V 10480 7500 50  0001 C CNN
-F 3 "~" H 10550 7500 50  0001 C CNN
-	1    10550 7500
-	1    0    0    -1
-$EndComp
-$Comp
-L Device:R R3
-U 1 1 5E84EE21
-P 10850 7500
-F 0 "R3" H 10920 7546 50  0000 L CNN
-F 1 "220" H 10920 7455 50  0000 L CNN
-F 2 "Resistor_SMD:R_0805_2012Metric" V 10780 7500 50  0001 C CNN
-F 3 "~" H 10850 7500 50  0001 C CNN
-	1    10850 7500
-	1    0    0    -1
-$EndComp
-$Comp
 L Device:R R5
 U 1 1 5E405AD0
@@
 	5250 9950 5600 9950
 $Comp
-L Connector:Bus_ISA_8bit X0
+L RTL8019-rescue:Bus_ISA_8bit-Connector X0
 U 1 1 5EAB26FD
 P 2500 2900
@@
 Text Label 6200 6700 0    50   ~ 0
 TPR-
+$Comp
+L Device:R R2
+U 1 1 5E84BDBA
+P 10550 7500
+F 0 "R2" H 10620 7546 50  0000 L CNN
+F 1 "510" H 10620 7455 50  0000 L CNN
+F 2 "Resistor_SMD:R_0805_2012Metric" V 10480 7500 50  0001 C CNN
+F 3 "~" H 10550 7500 50  0001 C CNN
+	1    10550 7500
+	1    0    0    -1
+$EndComp
+$Comp
+L Device:R R3
+U 1 1 5E84EE21
+P 10850 7500
+F 0 "R3" H 10920 7546 50  0000 L CNN
+F 1 "510" H 10920 7455 50  0000 L CNN
+F 2 "Resistor_SMD:R_0805_2012Metric" V 10780 7500 50  0001 C CNN
+F 3 "~" H 10850 7500 50  0001 C CNN
+	1    10850 7500
+	1    0    0    -1
+$EndComp
 $EndSCHEMATC
